Commit message: tag, box and search change

File: catkin_ws/src/manipulator-control/urdf/box.urdf.xacro (robot description, xacro)
@@ -1,11 +1,9 @@
 <?xml version="1.0"?>
 <robot name="box" xmlns:xacro="http://ros.org/wiki/xacro">
-  <link name="box_world"/>
-<!--Box with button-->
   <link name="box">
     <visual>
       <origin rpy="0 0 0" xyz="0 0 0"/>
       <geometry>
-        <mesh filename="package://manipulator-control/meshes/box.dae"/>
+        <box size="0.1 0.2 0.05"/>
       </geometry>
     </visual>
@@ -13,5 +11,5 @@
       <origin rpy="0 0 0" xyz="0 0 0"/>
       <geometry>
-        <mesh filename="package://manipulator-control/meshes/box.dae"/>
+        <box size="0.1 0.2 0.05"/>
       </geometry>
     </collision>
@@ -22,15 +20,10 @@
     </inertial>
   </link>
-  <joint name="box_joint" type="fixed">
-    <parent link="box_world"/>
-    <child link="box"/>
-    <!-- <origin rpy="0 0 3.14" xyz="-0.35 0 0.2"/> -->
-    <origin rpy="0 0 3.14" xyz="0 0 0"/>
-  </joint>
-  <link name="artag4">
+  <!-- Primeira caixa -->
+  <link name="artag1">
     <visual>
       <origin rpy="0 0 0" xyz="0 0 0"/>
       <geometry>
-        <mesh filename="package://manipulator-control/meshes/tag.dae"/>
+        <mesh filename="package://manipulator-control/meshes/tag.dae" scale="0.5 0.5 0.5"/>
       </geometry>
     </visual>
@@ -38,5 +31,5 @@
       <origin rpy="0 0 0" xyz="0 0 0"/>
       <geometry>
-        <mesh filename="package://manipulator-control/meshes/tag.dae"/>
+        <mesh filename="package://manipulator-control/meshes/tag.dae" scale="0.5 0.5 0.5"/>
       </geometry>
     </collision>
@@ -47,15 +40,58 @@
     </inertial>
   </link>
-  <joint name="tag_joint" type="fixed">
+  <joint name="tag_joint1" type="fixed">
     <parent link="box"/>
-    <child link="artag4"/>
-    <origin rpy="0 0 -1.571" xyz="0 0 0"/>
+    <child link="artag1"/>
+    <origin rpy="0 0 -1.571" xyz="-0.025 0.025 0.025"/>
   </joint>
-  <link name="button"/>
-  <joint name="button" type="fixed">
-    <parent link="artag4"/>
-    <child link="button"/>
-    <origin rpy="3.14 1.5708 3.14" xyz="0.12 0.0 0.07"/>
-    <!-- <origin rpy="0 0 0" xyz="0 -0.11500000 0.02361546"/> -->
+  <!-- Segunda caixa -->
+  <link name="artag2">
+    <visual>
+      <origin rpy="0 0 0" xyz="0 0 0"/>
+      <geometry>
+        <mesh filename="package://manipulator-control/meshes/tag.dae" scale="0.5 0.5 0.5"/>
+      </geometry>
+    </visual>
+    <collision>
+      <origin rpy="0 0 0" xyz="0 0 0"/>
+      <geometry>
+        <mesh filename="package://manipulator-control/meshes/tag.dae" scale="0.5 0.5 0.5"/>
+      </geometry>
+    </collision>
+    <inertial>
+      <origin rpy="0 0 0" xyz="0 0 0"/>
+      <mass value="0.01052000"/>
+      <inertia ixx="8.76754333e-6" ixy="0" ixz="0" iyx="0" iyy="8.76754333e-6" iyz="0" izx="0" izy="0" izz="1.75333333e-5"/>
+    </inertial>
+  </link>
+  <joint name="tag_joint2" type="fixed">
+    <parent link="box"/>
+    <child link="artag2"/>
+    <origin rpy="0 0 -1.571" xyz="-0.025 -0.025 0.025"/>
+  </joint>
+  <!-- Terceira caixa -->
+  <link name="artag3">
+    <visual>
+      <origin rpy="0 0 0" xyz="0 0 0"/>
+      <geometry>
+        <mesh filename="package://manipulator-control/meshes/tag.dae" scale="0.5 0.5 0.5"/>
+      </geometry>
+    </visual>
+    <collision>
+      <origin rpy="0 0 0" xyz="0 0 0"/>
+      <geometry>
+        <mesh filename="package://manipulator-control/meshes/tag.dae" scale="0.5 0.5 0.5"/>
+      </geometry>
+    </collision>
+    <inertial>
+      <origin rpy="0 0 0" xyz="0 0 0"/>
+      <mass value="0.01052000"/>
+      <inertia ixx="8.76754333e-6" ixy="0" ixz="0" iyx="0" iyy="8.76754333e-6" iyz="0" izx="0" izy="0" izz="1.75333333e-5"/>
+    </inertial>
+  </link>
+  <joint name="tag_joint3" type="fixed">
+    <parent link="box"/>
+    <child link="artag3"/>
+    <origin rpy="0 0 -1.571" xyz="0.025 0 0.025"/>
   </joint>
 </robot>

Commit message: tag

File: catkin_ws/src/manipulator-control/urdf/box.urdf.xacro (robot description, xacro)
@@ -1,4 +1,5 @@
 <?xml version="1.0"?>
 <robot name="box" xmlns:xacro="http://ros.org/wiki/xacro">
+  <xacro:property name="tag" value="tag.dae" />
   <link name="box">
     <visual>
@@ -25,5 +26,5 @@
       <origin rpy="0 0 0" xyz="0 0 0"/>
       <geometry>
-        <mesh filename="package://manipulator-control/meshes/tag.dae" scale="0.5 0.5 0.5"/>
+        <mesh filename="package://manipulator-control/meshes/${tag}" scale="0.5 0.5 0.5"/>
       </geometry>
     </visual>
@@ -31,5 +32,5 @@
       <origin rpy="0 0 0" xyz="0 0 0"/>
       <geometry>
-        <mesh filename="package://manipulator-control/meshes/tag.dae" scale="0.5 0.5 0.5"/>
+        <mesh filename="package://manipulator-control/meshes/${tag}" scale="0.5 0.5 0.5"/>
       </geometry>
     </collision>
@@ -50,5 +51,5 @@
       <origin rpy="0 0 0" xyz="0 0 0"/>
       <geometry>
-        <mesh filename="package://manipulator-control/meshes/tag.dae" scale="0.5 0.5 0.5"/>
+        <mesh filename="package://manipulator-control/meshes/${tag}" scale="0.5 0.5 0.5"/>
       </geometry>
     </visual>
@@ -56,5 +57,5 @@
       <origin rpy="0 0 0" xyz="0 0 0"/>
       <geometry>
-        <mesh filename="package://manipulator-control/meshes/tag.dae" scale="0.5 0.5 0.5"/>
+        <mesh filename="package://manipulator-control/meshes/${tag}" scale="0.5 0.5 0.5"/>
       </geometry>
     </collision>
@@ -75,5 +76,5 @@
       <origin rpy="0 0 0" xyz="0 0 0"/>
       <geometry>
-        <mesh filename="package://manipulator-control/meshes/tag.dae" scale="0.5 0.5 0.5"/>
+        <mesh filename="package://manipulator-control/meshes/${tag}" scale="0.5 0.5 0.5"/>
       </geometry>
     </visual>
@@ -81,5 +82,5 @@
       <origin rpy="0 0 0" xyz="0 0 0"/>
       <geometry>
-        <mesh filename="package://manipulator-control/meshes/tag.dae" scale="0.5 0.5 0.5"/>
+        <mesh filename="package://manipulator-control/meshes/${tag}" scale="0.5 0.5 0.5"/>
       </geometry>
     </collision>
