Commit message: funcionando garai

File: catkin_ws/src/open_manipulator_p_simulations/open_manipulator_p_gazebo/urdf/box.xacro (robot description, xacro)
@@ -2,4 +2,5 @@
 <robot name="box" xmlns:xacro="http://ros.org/wiki/xacro">
   <xacro:property name="tag" value="tag.dae" />
+  <!-- <link name="world"/> -->
   <link name="box">
     <visual>
@@ -26,5 +27,5 @@
       <origin rpy="0 0 0" xyz="0 0 0"/>
       <geometry>
-        <mesh filename="package://manipulator-control/meshes/${tag}" scale="0.5 0.5 0.5"/>
+        <mesh filename="package://manipulator-control/meshes/${tag}" scale="1 1 1"/>
       </geometry>
     </visual>
@@ -32,5 +33,5 @@
       <origin rpy="0 0 0" xyz="0 0 0"/>
       <geometry>
-        <mesh filename="package://manipulator-control/meshes/${tag}" scale="0.5 0.5 0.5"/>
+        <mesh filename="package://manipulator-control/meshes/${tag}" scale="1 1 1"/>
       </geometry>
     </collision>
@@ -47,5 +48,5 @@
   </joint>
   <!-- Segunda caixa -->
-  <link name="artag2">
+  <!-- <link name="artag2">
     <visual>
       <origin rpy="0 0 0" xyz="0 0 0"/>
@@ -70,7 +71,7 @@
     <child link="artag2"/>
     <origin rpy="0 0 -1.571" xyz="-0.025 -0.025 0.025"/>
-  </joint>
+  </joint> -->
   <!-- Terceira caixa -->
-  <link name="artag3">
+  <!-- <link name="artag3">
     <visual>
       <origin rpy="0 0 0" xyz="0 0 0"/>
@@ -95,4 +96,4 @@
     <child link="artag3"/>
     <origin rpy="0 0 -1.571" xyz="0.025 0 0.025"/>
-  </joint>
+  </joint> -->
 </robot>

Commit message: tag 50

File: catkin_ws/src/open_manipulator_p_simulations/open_manipulator_p_gazebo/urdf/box.xacro (robot description, xacro)
@@ -27,5 +27,5 @@
       <origin rpy="0 0 0" xyz="0 0 0"/>
       <geometry>
-        <mesh filename="package://manipulator-control/meshes/${tag}" scale="1 1 1"/>
+        <mesh filename="package://manipulator-control/meshes/${tag}" scale="0.5 0.5 0.5"/>
       </geometry>
     </visual>
@@ -33,5 +33,5 @@
       <origin rpy="0 0 0" xyz="0 0 0"/>
       <geometry>
-        <mesh filename="package://manipulator-control/meshes/${tag}" scale="1 1 1"/>
+        <mesh filename="package://manipulator-control/meshes/${tag}" scale="0.5 0.5 0.5"/>
       </geometry>
     </collision>
