Commit message: add cam to manipulator with gripper

File: catkin_ws/src/open_manipulator_p/open_manipulator_p_description/urdf/open_manipulator_p_with_gripper.urdf.xacro (robot description, xacro)
@@ -326,5 +326,5 @@
   </link>
   <!-- Realsense Camera Joint Position -->
-  <joint name="camera_joint" type="fixed">
+  <!-- <joint name="camera_joint" type="fixed">
     <axis xyz="0 1 0" />
     <origin xyz="0.070 0.032 0.052" rpy="0 0 0"/>
@@ -332,4 +332,68 @@
     <child link="camera_link"/>
   </joint>
-  <link name="camera_link"/>
+  <link name="camera_link"/> -->
+    <!-- Alterations of the urdf caso eu faça merda -->
+  <joint name="camera_joint" type="fixed">
+    <axis xyz="0 1 0" />
+    <origin xyz="0.075 -0.05 0.05" rpy="0 0 0"/>
+    <parent link="link6"/>
+    <child link="camera_link"/>
+  </joint>
+  <link name="camera_link">
+    <collision>
+      <origin xyz="0 0 0" rpy="0 0 0"/>
+      <geometry>
+    <box size="0.05 0.05 0.05"/>
+      </geometry>
+    </collision>
+    <visual>
+      <origin xyz="0 0 0" rpy="0 0 0"/>
+      <geometry>
+    <box size="0.05 0.05 0.05"/>
+      </geometry>
+      <material name="red"/>
+    </visual>
+    <inertial>
+      <mass value="1e-5" />
+      <origin xyz="0 0 0" rpy="0 0 0"/>
+      <inertia ixx="1e-6" ixy="0" ixz="0" iyy="1e-6" iyz="0" izz="1e-6" />
+    </inertial>
+  </link>
+  <!-- camera -->
+  <gazebo reference="camera_link">
+    <sensor type="camera" name="camera1">
+      <update_rate>30.0</update_rate>
+      <camera name="head">
+        <horizontal_fov>1.3962634</horizontal_fov>
+        <image>
+          <width>800</width>
+          <height>800</height>
+          <format>R8G8B8</format>
+        </image>
+        <clip>
+          <near>0.02</near>
+          <far>300</far>
+        </clip>
+        <noise>
+          <type>gaussian</type>
+          <mean>0.0</mean>
+          <stddev>0.007</stddev>
+        </noise>
+      </camera>
+      <plugin name="camera_controller" filename="libgazebo_ros_camera.so">
+        <alwaysOn>true</alwaysOn>
+        <updateRate>0.0</updateRate>
+        <cameraName>arm/camera1</cameraName>
+        <imageTopicName>image_raw</imageTopicName>
+        <cameraInfoTopicName>camera_info</cameraInfoTopicName>
+        <frameName>camera_link</frameName>
+        <hackBaseline>0.07</hackBaseline>
+        <distortionK1>0.0</distortionK1>
+        <distortionK2>0.0</distortionK2>
+        <distortionK3>0.0</distortionK3>
+        <distortionT1>0.0</distortionT1>
+        <distortionT2>0.0</distortionT2>
+      </plugin>
+    </sensor>
+  </gazebo>
 </robot>

Commit message: a

File: catkin_ws/src/open_manipulator_p/open_manipulator_p_description/urdf/open_manipulator_p_with_gripper.urdf.xacro (robot description, xacro)
@@ -397,3 +397,11 @@
     </sensor>
   </gazebo>
+  <!-- Fake camera link to reoriented the camera link -->
+  <link name="camera_fake"/>
+  <joint name="fake_joint" type="fixed">
+    <origin xyz="0 0 0" rpy="0 1.570796 0"/>
+    <parent link="camera_link"/>
+    <child link="camera_fake"/>
+  </joint>
+  <!-- 1.570796 -->
 </robot>
