Commit message: tryng to make joints work

File: catkin_ws/src/open_manipulator_p/open_manipulator_p_description/urdf/open_manipulator_p.urdf.xacro (robot description, xacro)
@@ -29,4 +29,5 @@
     <origin xyz="0.0 0.0 0.126" rpy="0 0 0"/>
     <axis xyz="0 0 1"/>
+    <!-- <limit velocity="6.5" effort="1000" lower="${-pi}" upper="${pi}" /> -->
     <limit velocity="6.5" effort="1000" lower="${-pi*0.5}" upper="${pi*0.5}" />
     <dynamics damping="0.7"/>
@@ -61,4 +62,5 @@
     <origin xyz="0.0 0.069 0.033" rpy="0 0 0"/>
     <axis xyz="0 1 0"/>
+    <!-- <limit velocity="6.5" effort="1000" lower="${-pi}" upper="${pi}" /> -->
     <limit velocity="6.5" effort="1000" lower="${-pi*0.5}" upper="${pi*0.5}" />
     <dynamics damping="0.7"/>

Commit message: cam working for real

File: catkin_ws/src/open_manipulator_p/open_manipulator_p_description/urdf/open_manipulator_p.urdf.xacro (robot description, xacro)
@@ -216,3 +216,68 @@
     </inertial>
   </link>
+  <!-- Alterations of the urdf caso eu faça merda -->
+  <!-- <xacro:property name="camera_link" value="0.05" /> Size of square 'camera' box -->
+  <joint name="camera_joint" type="fixed">
+    <axis xyz="0 1 0" />
+    <origin xyz="0.075 -0.05 0.05" rpy="0 0 0"/>
+    <parent link="link6"/>
+    <child link="camera_link"/>
+  </joint>
+  <link name="camera_link">
+    <collision>
+      <origin xyz="0 0 0" rpy="0 0 0"/>
+      <geometry>
+    <box size="0.05 0.05 0.05"/>
+      </geometry>
+    </collision>
+    <visual>
+      <origin xyz="0 0 0" rpy="0 0 0"/>
+      <geometry>
+    <box size="0.05 0.05 0.05"/>
+      </geometry>
+      <material name="red"/>
+    </visual>
+    <inertial>
+      <mass value="1e-5" />
+      <origin xyz="0 0 0" rpy="0 0 0"/>
+      <inertia ixx="1e-6" ixy="0" ixz="0" iyy="1e-6" iyz="0" izz="1e-6" />
+    </inertial>
+  </link>
+  <!-- camera -->
+  <gazebo reference="camera_link">
+    <sensor type="camera" name="camera1">
+      <update_rate>30.0</update_rate>
+      <camera name="head">
+        <horizontal_fov>1.3962634</horizontal_fov>
+        <image>
+          <width>800</width>
+          <height>800</height>
+          <format>R8G8B8</format>
+        </image>
+        <clip>
+          <near>0.02</near>
+          <far>300</far>
+        </clip>
+        <noise>
+          <type>gaussian</type>
+          <mean>0.0</mean>
+          <stddev>0.007</stddev>
+        </noise>
+      </camera>
+      <plugin name="camera_controller" filename="libgazebo_ros_camera.so">
+        <alwaysOn>true</alwaysOn>
+        <updateRate>0.0</updateRate>
+        <cameraName>arm/camera1</cameraName>
+        <imageTopicName>image_raw</imageTopicName>
+        <cameraInfoTopicName>camera_info</cameraInfoTopicName>
+        <frameName>camera_link</frameName>
+        <hackBaseline>0.07</hackBaseline>
+        <distortionK1>0.0</distortionK1>
+        <distortionK2>0.0</distortionK2>
+        <distortionK3>0.0</distortionK3>
+        <distortionT1>0.0</distortionT1>
+        <distortionT2>0.0</distortionT2>
+      </plugin>
+    </sensor>
+  </gazebo>
 </robot>

Commit message: correct joints

File: catkin_ws/src/open_manipulator_p/open_manipulator_p_description/urdf/open_manipulator_p.urdf.xacro (robot description, xacro)
@@ -60,8 +60,7 @@
     <parent link="link2"/>
     <child link="link3"/>
-    <origin xyz="0.0 0.069 0.033" rpy="0 0 0"/>
+<origin xyz="0.0 0.069 0.033" rpy="0 ${-pi} 0"/>
     <axis xyz="0 1 0"/>
-    <!-- <limit velocity="6.5" effort="1000" lower="${-pi}" upper="${pi}" /> -->
-    <limit velocity="6.5" effort="1000" lower="${-pi*0.5}" upper="${pi*0.5}" />
+    <limit velocity="6.5" effort="1000" lower="${-pi-pi*0.5}" upper="${-pi*0.5}" />
     <dynamics damping="0.7"/>
   </joint>
@@ -93,7 +92,7 @@
     <parent link="link3"/>
     <child link="link4"/>
-    <origin xyz="0.03000 -0.01150 0.26400" rpy="0 0 0"/>
+    <origin xyz="0.03000 -0.01150 0.26400" rpy="0 ${-pi*1.25} 0"/>
     <axis xyz="0 1 0"/>
-    <limit velocity="6.5" effort="1000" lower="${-pi*0.5}" upper="${pi*0.5}" />
+    <limit velocity="6.5" effort="1000" lower="${-pi*1.5}" upper="${-pi*0.25}" />
     <dynamics damping="0.7"/>
   </joint>
@@ -125,7 +124,7 @@
     <parent link="link4"/>
     <child link="link5"/>
-    <origin xyz="0.19500 -0.05750 0.03000" rpy="0 0 0"/>
+    <origin xyz="0.19500 -0.05750 0.03000" rpy="${-pi*0.5} 0 0"/>
     <axis xyz="1 0 0"/>
-    <limit velocity="6.5" effort="1000" lower="${-pi*0.5}" upper="${pi*0.5}" />
+    <limit velocity="6.5" effort="1000" lower="${-pi}" upper="${pi}" />
     <dynamics damping="0.7"/>
   </joint>
@@ -191,5 +190,5 @@
     <origin xyz="0.12300 -0.04500 0.00000" rpy="0 0 0"/>
     <axis xyz="1 0 0"/>
-    <limit velocity="6.5" effort="1000" lower="${-pi*0.5}" upper="${pi*0.5}" />
+    <limit velocity="6.5" effort="1000" lower="${-pi}" upper="${pi*0.5}" />
     <dynamics damping="0.7"/>
   </joint>

Commit message: aruco indentification

File: catkin_ws/src/open_manipulator_p/open_manipulator_p_description/urdf/open_manipulator_p.urdf.xacro (robot description, xacro)
@@ -280,3 +280,12 @@
     </sensor>
   </gazebo>
+  <!-- Fake camera link to reoriented the camera link -->
+  <link name="camera_fake"/>
+  <joint name="fake_joint" type="fixed">
+    <!-- <origin xyz="0 0 0" rpy="0 1.570796 0"/> -->
+    <origin xyz="0 0 0" rpy="1.5704 3.1416 1.5704"/>
+    <parent link="camera_link"/>
+    <child link="camera_fake"/>
+  </joint>
+  <!-- 1.570796 -->
 </robot>

Commit message: IS QUASE WORKING

File: catkin_ws/src/open_manipulator_p/open_manipulator_p_description/urdf/open_manipulator_p.urdf.xacro (robot description, xacro)
@@ -284,5 +284,5 @@
   <joint name="fake_joint" type="fixed">
     <!-- <origin xyz="0 0 0" rpy="0 1.570796 0"/> -->
-    <origin xyz="0 0 0" rpy="1.5704 3.1416 1.5704"/>
+    <origin xyz="0 0 0" rpy="1.5704 3.1416 3.1416"/>
     <parent link="camera_link"/>
     <child link="camera_fake"/>

Commit message: chages

File: catkin_ws/src/open_manipulator_p/open_manipulator_p_description/urdf/open_manipulator_p.urdf.xacro (robot description, xacro)
@@ -243,49 +243,13 @@
     </inertial>
   </link>
-  <!-- camera -->
-  <gazebo reference="camera_link">
-    <sensor type="camera" name="camera1">
-      <update_rate>30.0</update_rate>
-      <camera name="head">
-        <horizontal_fov>1.3962634</horizontal_fov>
-        <image>
-          <width>800</width>
-          <height>800</height>
-          <format>R8G8B8</format>
-        </image>
-        <clip>
-          <near>0.02</near>
-          <far>300</far>
-        </clip>
-        <noise>
-          <type>gaussian</type>
-          <mean>0.0</mean>
-          <stddev>0.007</stddev>
-        </noise>
-      </camera>
-      <plugin name="camera_controller" filename="libgazebo_ros_camera.so">
-        <alwaysOn>true</alwaysOn>
-        <updateRate>0.0</updateRate>
-        <cameraName>arm/camera1</cameraName>
-        <imageTopicName>image_raw</imageTopicName>
-        <cameraInfoTopicName>camera_info</cameraInfoTopicName>
-        <frameName>camera_link</frameName>
-        <hackBaseline>0.07</hackBaseline>
-        <distortionK1>0.0</distortionK1>
-        <distortionK2>0.0</distortionK2>
-        <distortionK3>0.0</distortionK3>
-        <distortionT1>0.0</distortionT1>
-        <distortionT2>0.0</distortionT2>
-      </plugin>
-    </sensor>
-  </gazebo>
   <!-- Fake camera link to reoriented the camera link -->
   <link name="camera_fake"/>
   <joint name="fake_joint" type="fixed">
     <!-- <origin xyz="0 0 0" rpy="0 1.570796 0"/> -->
-    <origin xyz="0 0 0" rpy="1.5704 3.1416 3.1416"/>
+    <origin xyz="0 0 0" rpy="${-pi/2} 0 0"/>
     <parent link="camera_link"/>
     <child link="camera_fake"/>
   </joint>
   <!-- 1.570796 -->
+  <!-- AAAAAAAAAAAAAAAAAAAAAAAAAAAAAAAAAAAAAAAAAAAAAAAAAAAAAAAAAAAAAAAAAAAAAAAAAAAAAAAAAAAAAAAA -->
 </robot>

Commit message: correcting commits

File: catkin_ws/src/open_manipulator_p/open_manipulator_p_description/urdf/open_manipulator_p.urdf.xacro (robot description, xacro)
@@ -60,8 +60,7 @@
     <parent link="link2"/>
     <child link="link3"/>
-    <origin xyz="0.0 0.069 0.033" rpy="0 0 0"/>
+<origin xyz="0.0 0.069 0.033" rpy="0 ${-pi} 0"/>
     <axis xyz="0 1 0"/>
-    <!-- <limit velocity="6.5" effort="1000" lower="${-pi}" upper="${pi}" /> -->
-    <limit velocity="6.5" effort="1000" lower="${-pi*0.5}" upper="${pi*0.5}" />
+    <limit velocity="6.5" effort="1000" lower="${-pi-pi*0.5}" upper="${-pi*0.5}" />
     <dynamics damping="0.7"/>
   </joint>
@@ -93,7 +92,7 @@
     <parent link="link3"/>
     <child link="link4"/>
-    <origin xyz="0.03000 -0.01150 0.26400" rpy="0 0 0"/>
+    <origin xyz="0.03000 -0.01150 0.26400" rpy="0 ${-pi*1.25} 0"/>
     <axis xyz="0 1 0"/>
-    <limit velocity="6.5" effort="1000" lower="${-pi*0.5}" upper="${pi*0.5}" />
+    <limit velocity="6.5" effort="1000" lower="${-pi*1.5}" upper="${-pi*0.25}" />
     <dynamics damping="0.7"/>
   </joint>
@@ -125,7 +124,7 @@
     <parent link="link4"/>
     <child link="link5"/>
-    <origin xyz="0.19500 -0.05750 0.03000" rpy="0 0 0"/>
+    <origin xyz="0.19500 -0.05750 0.03000" rpy="${-pi*0.5} 0 0"/>
     <axis xyz="1 0 0"/>
-    <limit velocity="6.5" effort="1000" lower="${-pi*0.5}" upper="${pi*0.5}" />
+    <limit velocity="6.5" effort="1000" lower="${-pi}" upper="${pi}" />
     <dynamics damping="0.7"/>
   </joint>
@@ -191,5 +190,5 @@
     <origin xyz="0.12300 -0.04500 0.00000" rpy="0 0 0"/>
     <axis xyz="1 0 0"/>
-    <limit velocity="6.5" effort="1000" lower="${-pi*0.5}" upper="${pi*0.5}" />
+    <limit velocity="6.5" effort="1000" lower="${-pi}" upper="${pi*0.5}" />
     <dynamics damping="0.7"/>
   </joint>
@@ -244,40 +243,13 @@
     </inertial>
   </link>
-  <!-- camera -->
-  <gazebo reference="camera_link">
-    <sensor type="camera" name="camera1">
-      <update_rate>30.0</update_rate>
-      <camera name="head">
-        <horizontal_fov>1.3962634</horizontal_fov>
-        <image>
-          <width>800</width>
-          <height>800</height>
-          <format>R8G8B8</format>
-        </image>
-        <clip>
-          <near>0.02</near>
-          <far>300</far>
-        </clip>
-        <noise>
-          <type>gaussian</type>
-          <mean>0.0</mean>
-          <stddev>0.007</stddev>
-        </noise>
-      </camera>
-      <plugin name="camera_controller" filename="libgazebo_ros_camera.so">
-        <alwaysOn>true</alwaysOn>
-        <updateRate>0.0</updateRate>
-        <cameraName>arm/camera1</cameraName>
-        <imageTopicName>image_raw</imageTopicName>
-        <cameraInfoTopicName>camera_info</cameraInfoTopicName>
-        <frameName>camera_link</frameName>
-        <hackBaseline>0.07</hackBaseline>
-        <distortionK1>0.0</distortionK1>
-        <distortionK2>0.0</distortionK2>
-        <distortionK3>0.0</distortionK3>
-        <distortionT1>0.0</distortionT1>
-        <distortionT2>0.0</distortionT2>
-      </plugin>
-    </sensor>
-  </gazebo>
+  <!-- Fake camera link to reoriented the camera link -->
+  <link name="camera_fake"/>
+  <joint name="fake_joint" type="fixed">
+    <!-- <origin xyz="0 0 0" rpy="0 1.570796 0"/> -->
+    <origin xyz="0 0 0" rpy="${-pi/2} 0 0"/>
+    <parent link="camera_link"/>
+    <child link="camera_fake"/>
+  </joint>
+  <!-- 1.570796 -->
+  <!-- AAAAAAAAAAAAAAAAAAAAAAAAAAAAAAAAAAAAAAAAAAAAAAAAAAAAAAAAAAAAAAAAAAAAAAAAAAAAAAAAAAAAAAAA -->
 </robot>

Commit message: a

File: catkin_ws/src/open_manipulator_p/open_manipulator_p_description/urdf/open_manipulator_p.urdf.xacro (robot description, xacro)
@@ -247,5 +247,5 @@
   <joint name="fake_joint" type="fixed">
     <!-- <origin xyz="0 0 0" rpy="0 1.570796 0"/> -->
-    <origin xyz="0 0 0" rpy="${-pi/2} 0 0"/>
+    <origin xyz="0 0 0" rpy="${pi/2} 0 0"/>
     <parent link="camera_link"/>
     <child link="camera_fake"/>

Commit message: quase last commit

File: catkin_ws/src/open_manipulator_p/open_manipulator_p_description/urdf/open_manipulator_p.urdf.xacro (robot description, xacro)
@@ -62,5 +62,5 @@
 <origin xyz="0.0 0.069 0.033" rpy="0 ${-pi} 0"/>
     <axis xyz="0 1 0"/>
-    <limit velocity="6.5" effort="1000" lower="${-pi-pi*0.5}" upper="${-pi*0.5}" />
+    <limit velocity="6.5" effort="1000" lower="${-pi*1.5}" upper="${-pi*0.5}" />
     <dynamics damping="0.7"/>
   </joint>
@@ -158,5 +158,5 @@
     <origin xyz="0.06300 0.04500 0.00000" rpy="0 0 0"/>
     <axis xyz="0 1 0"/>
-    <limit velocity="6.5" effort="1000" lower="${-pi*0.5}" upper="${pi*0.5}" />
+    <limit velocity="6.5" effort="1000" lower="${-pi*70/180}" upper="${pi*70/180}" />
     <dynamics damping="0.7"/>
   </joint>
@@ -190,5 +190,5 @@
     <origin xyz="0.12300 -0.04500 0.00000" rpy="0 0 0"/>
     <axis xyz="1 0 0"/>
-    <limit velocity="6.5" effort="1000" lower="${-pi}" upper="${pi*0.5}" />
+    <limit velocity="6.5" effort="1000" lower="${-pi*170/180}" upper="${0}" />
     <dynamics damping="0.7"/>
   </joint>

Commit message: first commit

File: catkin_ws/src/open_manipulator_p/open_manipulator_p_description/urdf/open_manipulator_p.urdf.xacro (robot description, xacro)
@@ -60,7 +60,8 @@
     <parent link="link2"/>
     <child link="link3"/>
-<origin xyz="0.0 0.069 0.033" rpy="0 ${-pi} 0"/>
+    <origin xyz="0.0 0.069 0.033" rpy="0 0 0"/>
     <axis xyz="0 1 0"/>
-    <limit velocity="6.5" effort="1000" lower="${-pi*1.5}" upper="${-pi*0.5}" />
+    <!-- <limit velocity="6.5" effort="1000" lower="${-pi}" upper="${pi}" /> -->
+    <limit velocity="6.5" effort="1000" lower="${-pi*0.5}" upper="${pi*0.5}" />
     <dynamics damping="0.7"/>
   </joint>
@@ -92,7 +93,7 @@
     <parent link="link3"/>
     <child link="link4"/>
-    <origin xyz="0.03000 -0.01150 0.26400" rpy="0 ${-pi*1.25} 0"/>
+    <origin xyz="0.03000 -0.01150 0.26400" rpy="0 0 0"/>
     <axis xyz="0 1 0"/>
-    <limit velocity="6.5" effort="1000" lower="${-pi*1.5}" upper="${-pi*0.25}" />
+    <limit velocity="6.5" effort="1000" lower="${-pi*0.5}" upper="${pi*0.5}" />
     <dynamics damping="0.7"/>
   </joint>
@@ -124,7 +125,7 @@
     <parent link="link4"/>
     <child link="link5"/>
-    <origin xyz="0.19500 -0.05750 0.03000" rpy="${-pi*0.5} 0 0"/>
+    <origin xyz="0.19500 -0.05750 0.03000" rpy="0 0 0"/>
     <axis xyz="1 0 0"/>
-    <limit velocity="6.5" effort="1000" lower="${-pi}" upper="${pi}" />
+    <limit velocity="6.5" effort="1000" lower="${-pi*0.5}" upper="${pi*0.5}" />
     <dynamics damping="0.7"/>
   </joint>
@@ -158,5 +159,5 @@
     <origin xyz="0.06300 0.04500 0.00000" rpy="0 0 0"/>
     <axis xyz="0 1 0"/>
-    <limit velocity="6.5" effort="1000" lower="${-pi*70/180}" upper="${pi*70/180}" />
+    <limit velocity="6.5" effort="1000" lower="${-pi*0.5}" upper="${pi*0.5}" />
     <dynamics damping="0.7"/>
   </joint>
@@ -190,5 +191,5 @@
     <origin xyz="0.12300 -0.04500 0.00000" rpy="0 0 0"/>
     <axis xyz="1 0 0"/>
-    <limit velocity="6.5" effort="1000" lower="${-pi*170/180}" upper="${0}" />
+    <limit velocity="6.5" effort="1000" lower="${-pi*0.5}" upper="${pi*0.5}" />
     <dynamics damping="0.7"/>
   </joint>
